File: pcb/momo_modular/controller/controller.brd (EAGLE design)
At the start: 19 parts, among them U6 PIC24F16KA101-X_PSSOP, U7 FLASH8MSOP8

Commit message: Added latest pcb file versions
Parts:
- moved C1 0.21 mm to (46.8, 26.1)
Routing:
- net GND: track 105.6 -> 104.5 mm
- net N$25: track 6.85 -> 7.45 mm
- net N$3: track 3.75 -> 3.16 mm
