File: pcb/momo_modular/controller_wallpower/wall_power.brd (EAGLE design)
At the start: 34.1 x 33 mm, 30 parts, among them U1 XRP7659, U2 MCP1702, U3 PIC24F16KA101-X_PSSOP, U4 FLASH8MSOP8

Commit message: Final wallpower board changes
Parts:
- C5: value 22 uF -> 1 uF
Changed lines of the file:
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@@
 <attribute name="VALUE" x="51.1048" y="24.0538" size="1.27" layer="27" rot="R180"/>
 </element>
-<element name="C5" library="rcl" package="C0402" value="22 uF" x="49.5046" y="23.4188" smashed="yes">
+<element name="C5" library="rcl" package="C0402" value="1 uF" x="49.5046" y="23.4188" smashed="yes">
 <attribute name="NAME" x="50.292" y="23.0632" size="0.8128" layer="25"/>
 <attribute name="VALUE" x="48.8696" y="21.5138" size="1.27" layer="27"/>
@@
 </signal>
 </signals>
-<errors>
-</errors>
 </board>
 </drawing>
