File: pcb/momo_modular/controller_wallpower/wall_power.sch (EAGLE design)
At the start: 30 parts, among them U1 XRP7659, U2 MCP1702, U3 PIC24F16KA101-X_PSSOP, U4 FLASH8MSOP8

Commit message: Final wallpower board changes
Parts:
- C5: value 22 uF -> 1 uF
Changed lines of the file:
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@@
 <part name="GND8" library="supply1" deviceset="GND" device=""/>
 <part name="U2" library="components" deviceset="MCP1702" device=""/>
-<part name="C5" library="rcl" deviceset="C-US" device="C0402" value="22 uF"/>
+<part name="C5" library="rcl" deviceset="C-US" device="C0402" value="1 uF"/>
 <part name="GND11" library="supply1" deviceset="GND" device=""/>
 <part name="GND12" library="supply1" deviceset="GND" device=""/>
