File: pcb/momo_modular/sensor_elec_sd/sensor_elec_sd.sch (EAGLE design)
At the start: 27 parts, among them U1 AP7115-LDO, U2 16LF1847, U3 TS1100

Commit message: Added global attributes to board to work with production building scripts
Parts:
- JP2: DIGIKEY-PN (none) -> S7004-ND
Changed lines of the file:
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@@
 <setting verticaltext="up"/>
 </settings>
-<grid distance="0.1" unitdist="inch" unit="inch" style="lines" multiple="4" display="no" altdistance="0.01" altunitdist="inch" altunit="inch"/>
+<grid distance="0.1" unitdist="inch" unit="inch" style="lines" multiple="1" display="no" altdistance="0.01" altunitdist="inch" altunit="inch"/>
 <layers>
 <layer number="1" name="Top" color="4" fill="1" visible="no" active="no"/>
@@
 <attribute name="DIGIKEY-PN" value="P10KGCT-ND"/>
 </part>
-<part name="JP2" library="components" deviceset="MOMO-VERT-6M" device=""/>
+<part name="JP2" library="components" deviceset="MOMO-VERT-6M" device="">
+<attribute name="DIGIKEY-PN" value="S7004-ND"/>
+</part>
 <part name="P+2" library="supply1" deviceset="V+" device=""/>
 <part name="VCC4" library="supply1" deviceset="VCCINT" device=""/>
@@
 <attribute name="DIGIKEY-PN" x="15.24" y="17.78" size="1.778" layer="96" rot="R90" display="off"/>
 </instance>
-<instance part="JP2" gate="G$1" x="-86.36" y="-15.24"/>
+<instance part="JP2" gate="G$1" x="-86.36" y="-15.24">
+<attribute name="DIGIKEY-PN" x="-86.36" y="-15.24" size="1.778" layer="96" display="off"/>
+</instance>
 <instance part="P+2" gate="1" x="-78.74" y="7.62"/>
 <instance part="VCC4" gate="G$1" x="-81.28" y="7.62"/>

Commit message: Final changes to sd card and voltage sensing board.
Parts:
- added JP6: (no value), pinhead:PINHD-1X1
Connections:
- net N$4: now also JP6.1
Other:
- note added: "Programming Header"
Changed lines of the file:
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@@
 <part name="JP4" library="components" deviceset="MOMO-SENSOR-RJ11" device=""/>
 <part name="JP5" library="components" deviceset="SCREWTERM4" device=""/>
+<part name="JP6" library="pinhead" deviceset="PINHD-1X1" device=""/>
 </parts>
 <sheets>
@@
 <text x="-103.632" y="-93.726" size="1.778" layer="97">1.0</text>
 <text x="-103.632" y="-96.266" size="1.778" layer="97">11/6/2013</text>
+<text x="40.64" y="25.4" size="1.778" layer="97">Programming Header</text>
 </plain>
 <instances>
@@
 <instance part="JP4" gate="G$1" x="-60.96" y="-12.7" rot="R180"/>
 <instance part="JP5" gate="G$1" x="-101.6" y="-40.64" rot="R180"/>
+<instance part="JP6" gate="G$1" x="38.1" y="25.4"/>
 </instances>
 <busses>
@@
 <pinref part="R1" gate="G$1" pin="1"/>
 <wire x1="15.24" y1="10.16" x2="15.24" y2="12.7" width="0.1524" layer="91"/>
-</segment>
-</net>
+<wire x1="15.24" y1="12.7" x2="30.48" y2="12.7" width="0.1524" layer="91"/>
+<wire x1="30.48" y1="12.7" x2="30.48" y2="25.4" width="0.1524" layer="91"/>
+<junction x="15.24" y="12.7"/>
+<pinref part="JP6" gate="G$1" pin="1"/>
+<wire x1="30.48" y1="25.4" x2="35.56" y2="25.4" width="0.1524" layer="91"/>
+</segment>
+</net>

Commit message: Finished divider network spec'ing and standardized on 1% resistors to reduce BOM lines.
Parts:
- C5: DIGIKEY-PN (none) -> 445-1265-1-ND; DIGKIEY-PN 445-1265-1-ND -> (none)
- R1: DIGIKEY-PN P10KGCT-ND -> P10.0KHCT-ND
- R11: DIGIKEY-PN P100KGCT-ND -> P100KHCT-ND
- R2: DIGIKEY-PN (none) -> CRF2512-FV-R001ELFCT-ND; DIGKEY-PN CRF2512-FV-R001ELFCT-ND -> (none)
- R3, R5: value (none) -> 620K 1%; DIGIKEY-PN (none) -> P620KHCT-ND
- R4, R6, R8: value (none) -> 100K 1%; DIGIKEY-PN (none) -> P100KHCT-ND
- R7: value (none) -> 806K 1%; DIGIKEY-PN (none) -> P806KHCT-ND
Changed lines of the file:
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@@
 <part name="VCC3" library="supply1" deviceset="VCCINT" device=""/>
 <part name="R1" library="rcl" deviceset="R-US_" device="R0603" value="10K">
-<attribute name="DIGIKEY-PN" value="P10KGCT-ND"/>
+<attribute name="DIGIKEY-PN" value="P10.0KHCT-ND"/>
 </part>
 <part name="JP2" library="components" deviceset="MOMO-VERT-6M" device="">
@@
 <part name="U3" library="components" deviceset="TS1100" device=""/>
 <part name="R2" library="rcl" deviceset="R-US_" device="R2512" value="0.001R">
-<attribute name="DIGKEY-PN" value="CRF2512-FV-R001ELFCT-ND"/>
+<attribute name="DIGIKEY-PN" value="CRF2512-FV-R001ELFCT-ND"/>
 </part>
 <part name="GND5" library="supply1" deviceset="GND" device=""/>
@@
 <part name="JP3" library="components" deviceset="5MM-SCREWTERM-2POS" device=""/>
 <part name="C5" library="rcl" deviceset="C-US" device="C0402K" value="100 nF">
-<attribute name="DIGKIEY-PN" value="445-1265-1-ND"/>
+<attribute name="DIGIKEY-PN" value="445-1265-1-ND"/>
 </part>
 <part name="GND7" library="supply1" deviceset="GND" device=""/>
 <part name="VCC5" library="supply1" deviceset="VCCINT" device=""/>
-<part name="R3" library="rcl" deviceset="R-US_" device="R0603"/>
-<part name="R4" library="rcl" deviceset="R-US_" device="R0603"/>
-<part name="R5" library="rcl" deviceset="R-US_" device="R0603"/>
-<part name="R6" library="rcl" deviceset="R-US_" device="R0603"/>
-<part name="R7" library="rcl" deviceset="R-US_" device="R0603"/>
-<part name="R8" library="rcl" deviceset="R-US_" device="R0603"/>
+<part name="R3" library="rcl" deviceset="R-US_" device="R0603" value="620K 1%">
+<attribute name="DIGIKEY-PN" value="P620KHCT-ND"/>
+</part>
+<part name="R4" library="rcl" deviceset="R-US_" device="R0603" value="100K 1%">
+<attribute name="DIGIKEY-PN" value="P100KHCT-ND"/>
+</part>
+<part name="R5" library="rcl" deviceset="R-US_" device="R0603" value="620K 1%">
+<attribute name="DIGIKEY-PN" value="P620KHCT-ND"/>
+</part>
+<part name="R6" library="rcl" deviceset="R-US_" device="R0603" value="100K 1%">
+<attribute name="DIGIKEY-PN" value="P100KHCT-ND"/>
+</part>
+<part name="R7" library="rcl" deviceset="R-US_" device="R0603" value="806K 1%">
+<attribute name="DIGIKEY-PN" value="P806KHCT-ND"/>
+</part>
+<part name="R8" library="rcl" deviceset="R-US_" device="R0603" value="100K 1%">
+<attribute name="DIGIKEY-PN" value="P100KHCT-ND"/>
+</part>
 <part name="C6" library="rcl" deviceset="C-US" device="C0402K" value="100 nF">
 <attribute name="DIGIKEY-PN" value="445-1265-1-ND"/>
@@
 <part name="GND12" library="supply1" deviceset="GND" device=""/>
 <part name="R11" library="rcl" deviceset="R-US_" device="R0603" value="100K">
-<attribute name="DIGIKEY-PN" value="P100KGCT-ND"/>
+<attribute name="DIGIKEY-PN" value="P100KHCT-ND"/>
 </part>
 <part name="GND9" library="supply1" deviceset="GND" device=""/>
@@
 <instance part="U3" gate="G$1" x="-78.74" y="45.72"/>
 <instance part="R2" gate="G$1" x="-76.2" y="66.04">
-<attribute name="DIGKEY-PN" x="-76.2" y="66.04" size="1.778" layer="96" display="off"/>
+<attribute name="DIGIKEY-PN" x="-76.2" y="66.04" size="1.778" layer="96" display="off"/>
 </instance>
 <instance part="GND5" gate="1" x="-76.2" y="33.02"/>
@@
 <instance part="JP3" gate="G$1" x="-55.88" y="73.66"/>
 <instance part="C5" gate="G$1" x="-2.54" y="68.58">
-<attribute name="DIGKIEY-PN" x="-2.54" y="68.58" size="1.778" layer="96" display="off"/>
+<attribute name="DIGIKEY-PN" x="-2.54" y="68.58" size="1.778" layer="96" display="off"/>
 </instance>
 <instance part="GND7" gate="1" x="-2.54" y="60.96"/>
 <instance part="VCC5" gate="G$1" x="-2.54" y="73.66"/>
-<instance part="R3" gate="G$1" x="-88.9" y="-55.88" rot="R90"/>
-<instance part="R4" gate="G$1" x="-88.9" y="-66.04" rot="R90"/>
-<instance part="R5" gate="G$1" x="-73.66" y="-55.88" rot="R90"/>
-<instance part="R6" gate="G$1" x="-73.66" y="-66.04" rot="R90"/>
-<instance part="R7" gate="G$1" x="-58.42" y="-55.88" rot="R90"/>
-<instance part="R8" gate="G$1" x="-58.42" y="-66.04" rot="R90"/>
+<instance part="R3" gate="G$1" x="-88.9" y="-55.88" rot="R90">
+<attribute name="DIGIKEY-PN" x="-88.9" y="-55.88" size="1.778" layer="96" rot="R90" display="off"/>
+</instance>
+<instance part="R4" gate="G$1" x="-88.9" y="-66.04" rot="R90">
+<attribute name="DIGIKEY-PN" x="-88.9" y="-66.04" size="1.778" layer="96" rot="R90" display="off"/>
+</instance>
+<instance part="R5" gate="G$1" x="-73.66" y="-55.88" rot="R90">
+<attribute name="DIGIKEY-PN" x="-73.66" y="-55.88" size="1.778" layer="96" rot="R90" display="off"/>
+</instance>
+<instance part="R6" gate="G$1" x="-73.66" y="-66.04" rot="R90">
+<attribute name="DIGIKEY-PN" x="-73.66" y="-66.04" size="1.778" layer="96" rot="R90" display="off"/>
+</instance>
+<instance part="R7" gate="G$1" x="-58.42" y="-55.88" rot="R90">
+<attribute name="DIGIKEY-PN" x="-58.42" y="-55.88" size="1.778" layer="96" rot="R90" display="off"/>
+</instance>
+<instance part="R8" gate="G$1" x="-58.42" y="-66.04" rot="R90">
+<attribute name="DIGIKEY-PN" x="-58.42" y="-66.04" size="1.778" layer="96" rot="R90" display="off"/>
+</instance>
 <instance part="C6" gate="G$1" x="-83.82" y="-66.04">
 <attribute name="DIGIKEY-PN" x="-83.82" y="-66.04" size="1.778" layer="96" display="off"/>
